File: Hardware/asic_board.kicad_sch (KiCad schematic)
At the start: 30 parts, among them J201 Conn_02x20_Odd_Even, J202 Keyboard, J203 Edge_Connector, U201 MegaDuck_Interface_CPU, U202 74LS241, U203 by ManCloud, Y201 Crystal

Commit message: Finished work on Mainboard
* Complete reversed Schematic incl. Signal "assumptions"
* Complete traced MainBoard-PCB
Parts:
- J201: footprint (none) -> Connector_PinHeader_2.54mm:PinHeader_2x20_P2.54mm_Vertical
Changed lines of the file:
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@@
 			)
 		)
-		(property "Footprint" ""
+		(property "Footprint" "Connector_PinHeader_2.54mm:PinHeader_2x20_P2.54mm_Vertical"
 			(at 80.01 233.68 0)
 			(effects
