File: Hardware/mainboard.kicad_sch (KiCad schematic)
At the start: 99 parts, among them J101 ProgrammCard, J102 MemoryCard, J103 Edge_Connector, J104 LCD_CON, J105 LINK_PORT, J106 EXT_AUDIO, J107 MOUSE_PORT, J108 Voice_Board_Mock, Q101 C9012, U101 MegaDuck_CPU, U102 GM76C88LFW-15, U103 GM76C88LFW-15, U104 LM386, U105 LM324, U106 CD4066BE, U107 CD4066BE, U108 74HC00, U109 74LS32, U110 74LS174, U111 27C040, U112 by ManCloud, Y101 4.194304MHz

Commit message: Finished work on Mainboard
* Complete reversed Schematic incl. Signal "assumptions"
* Complete traced MainBoard-PCB
Parts:
- added C12: 10n, symbol Device:C
- added R132, R133: NP, Resistor_SMD:R_0805_2012Metric, symbol Device:R
- added TP101, TP102: TestPoint, TestPoint:TestPoint_Pad_D1.5mm, symbol Connector:TestPoint
- added U113: LM324, Package_DIP:DIP-14_W7.62mm, symbol Amplifier_Operational:LM324
- C101, C110: value ?u -> 220u; footprint (none) -> Capacitor_THT:CP_Radial_D6.3mm_P2.50mm
- C102, C103, C104, C105, C106, C107: value ?u -> 1u; footprint (none) -> Capacitor_THT:CP_Radial_D5.0mm_P2.50mm
- C108, C109, C111: value ?u -> 10u; footprint (none) -> Capacitor_THT:CP_Radial_D4.0mm_P2.00mm
- C112: value ?u -> 470u; footprint (none) -> Capacitor_THT:CP_Radial_D6.3mm_P2.50mm
- C113, C114: value C -> 27p; footprint (none) -> Capacitor_SMD:C_0805_2012Metric
- C115, C116, C117, C118, C119, C120, C121: value C -> 100n; footprint (none) -> Capacitor_SMD:C_0805_2012Metric
- D101: footprint Diode_THT:D_DO-41_SOD81_P10.16mm_Horizontal -> Diode_THT:D_A-405_P7.62mm_Horizontal
- FB101, FB102, FB103, FB104, FB105, FB106, FB107, FB108, FB109, FB110, FB111, FB112, FB113, FB114: footprint (none) -> Inductor_THT:L_Axial_L5.3mm_D2.2mm_P2.54mm_Vertical_Vishay_IM-1
- J101, J102: footprint (none) -> Eigene:Edge-Cart-Connector_2x18_P2.54mm_Horizontal
- J103: footprint (none) -> MegaDuck:Edge_Connector
- J104: footprint (none) -> Connector_PinHeader_2.54mm:PinHeader_2x08_P2.54mm_Horizontal
- J105: footprint (none) -> Connector_PinHeader_2.54mm:PinHeader_1x03_P2.54mm_Vertical
- J106: footprint (none) -> Connector_PinHeader_2.54mm:PinHeader_1x05_P2.54mm_Vertical
- J107: footprint (none) -> MegaDuck:Mouse_Connector
- J108: footprint (none) -> MegaDuck:MD_VoiceChip
- Q101: footprint (none) -> Package_TO_SOT_THT:TO-92_Inline_Wide
- R101: value R -> 2k2; footprint (none) -> Resistor_SMD:R_0805_2012Metric
- R102: value R -> 1M; footprint (none) -> Resistor_SMD:R_0805_2012Metric
- R103, R104, R105, R107: value R -> 220; footprint (none) -> Resistor_SMD:R_0805_2012Metric
- R106, R110, R115, R131: value R -> 47k; footprint (none) -> Resistor_SMD:R_0805_2012Metric
- R108, R126, R127, R128: value R -> 4k7; footprint (none) -> Resistor_SMD:R_0805_2012Metric
- R109, R116, R117, R118, R121: value R -> 10k; footprint (none) -> Resistor_SMD:R_0805_2012Metric
- R111, R114, R130: value R -> 680; footprint (none) -> Resistor_SMD:R_0805_2012Metric
- R112, R113, R125: value R -> 100k; footprint (none) -> Resistor_SMD:R_0805_2012Metric
- R119: value R -> 1M2; footprint (none) -> Resistor_SMD:R_0805_2012Metric
- R120: value R -> 560k; footprint (none) -> Resistor_SMD:R_0805_2012Metric
- R122: value R -> 330k; footprint (none) -> Resistor_SMD:R_0805_2012Metric
- R123: value R -> 10M; footprint (none) -> Resistor_SMD:R_0805_2012Metric
- R124: value R -> 15k; footprint (none) -> Resistor_SMD:R_0805_2012Metric
- R129: value R -> 180k; footprint (none) -> Resistor_SMD:R_0805_2012Metric
- RV101: value R_Potentiometer -> 75k; footprint (none) -> Potentiometer_THT:Potentiometer_Bourns_3296W_Vertical
- U101: value MegaDuck_CPU -> DMG CPU
- U102, U103: footprint Gekkio_GameBoy:SOP-28_8.6x18mm_Pitch1.27mm -> Gekkio_Package_SO:Sharp_SOIC-28W_8.6x18mm_P1.27mm
- U104: footprint (none) -> Package_DIP:DIP-8_W7.62mm
- U105: footprint (none) -> Package_SO:SOIC-14_3.9x8.7mm_P1.27mm
- U108, U109: footprint (none) -> Package_DIP:DIP-14_W7.62mm
- U110: footprint (none) -> Package_DIP:DIP-16_W7.62mm
- U111: footprint (none) -> Package_DIP:DIP-32_W15.24mm
- Y101: footprint (none) -> Crystal:Crystal_HC18-U_Horizontal
Connections:
- net MC_?_0 is gone; now on net P12: J102.30 (Pin_30)
- net MC_?_1 is gone; now on net P14: J102.31 (Pin_31)
- net MC_?_2 is gone; now on net EDGE_31: J102.32 (Pin_32)
- net PC_?_0 is gone; now on net PHI: J101.2 (Pin_2)
- net PC_?_1 is gone; now on net ~{CS}: J101.5 (Pin_5)
- net PC_?_2 is gone; now on net VIN: J101.31 (Pin_31)
- net VCC is gone; now on net VDD: J101.1 (Pin_1), J102.1 (Pin_1), U101.58 (VDD)
- net ~{RST} is gone; now on net ~{RES}: J101.30 (Pin_30), U101.71 (~{RES})
- net A0: now also U103.10 (A0), U111.12 (A0)
- net A1: now also U103.9 (A1), U111.11 (A1)
- net A10: now also U103.21 (A10), U111.23 (A10)
- net A11: now also U103.23 (A11), U111.25 (A11)
- net A12: now also U103.2 (A12), U111.4 (A12)
- net A13: now also U109.13, U111.28 (A13)
- net A14: now also D108.2 (A), U103.26 (CE2), U109.9, U111.29 (A14)
- net A15: now also U108.1, U108.2; no longer J101.21 (Pin_21)
- net A2: now also U103.8 (A2), U111.10 (A2)
- net A3: now also U103.7 (A3), U111.9 (A3)
- net A4: now also U103.6 (A4), U111.8 (A4)
- net A5: now also U103.5 (A5), U111.7 (A5)
- net A6: now also U103.4 (A6), U111.6 (A6)
- net A7: now also U103.3 (A7), U111.5 (A7)
- net A8: now also U103.25 (A8), U111.27 (A8)
- net A9: now also U103.24 (A9), U111.26 (A9)
- net CART_SENSE: now also J103.32 (Pin_32)
- net D0: now also U103.11 (I/O0), U110.3 (D0), U111.13 (D0)
- net D1: now also U103.12 (I/O1), U110.4 (D1), U111.14 (D1)
- net D2: now also U103.13 (I/O2), U110.6 (D2), U111.15 (D2)
- net D3: now also U103.15 (I/O3), U110.11 (D3), U111.17 (D3)
- net D4: now also U103.16 (I/O4), U110.13 (D4), U111.18 (D4)
- net D5: now also U103.17 (I/O5), U110.14 (D5), U111.19 (D5)
- net D6: now also U103.18 (I/O6), U111.20 (D6)
- net D7: now also U103.19 (I/O7), U111.21 (D7)
- net GND: now also C101.2, C108.2, C109.2, C111.2, C112.2, C113.2, C114.2, C115.2, C116.2, C120.1, C121.2, D110.1 (K), FB101.1, FB101.2, FB102.1, FB102.2, FB107.1, FB107.2, FB111.1, FB111.2, FB114.1, FB114.2, J103.1 (Pin_1), J103.33 (Pin_33), J103.34 (Pin_34), J104.16 (Pin_16), J106.2 (Pin_2), J108.1 (Pin_1), R109.1, R117.2, R121.2, R125.2, R128.2, R130.2, RV101.3, U101.76 (T2), U101.77 (T1), U102.14 (GND), U103.14 (GND), U104.2 (-), U104.4 (GND), U105.11 (V-), U106.7 (V_{SS}), U107.7 (V_{SS}), U108.7 (GND), U109.7 (GND), U110.8 (GND), U111.16 (GND), C12.2, U113.11 (V-)
- net MC_?_3: now also R110.2, R112.1, U105.2 (-), R132.1, U113.2 (-)
- net MC_?_4: now also U105.6 (-), U113.6 (-)
- net MC_?_5: now also R125.1, U109.2, U109.4
- net SRAM_A13: now also U110.12 (Q4)
- net SRAM_A14: now also U110.15 (Q5)
- net ~{CS}: now also D107.2 (A), U103.20 (~{CE1}); no longer J102.29 (Pin_29)
- net ~{RD}: now also U103.22 (~{OE}), U111.24 (~{OE})
- net ~{WR}: now also U103.27 (~{WE}), U109.12
- net at R112.2: now also C104.1, U105.1, U113.1
- net at U109.10: now also U109.11
- net MAPPER_CLK: now reaches U109.8
- net MAPPER_CLK: now also U110.9 (Cp)
- net at C103.1: now also R132.2
- net SO2: now reaches C103.2
- net SO2: now also U101.59 (SO2)
- net XTAL_1: now reaches C113.1
- net XTAL_1: now also C117.2, J103.29 (Pin_29), R102.1, Y101.2
- net S: now reaches J104.1 (Pin_1)
- net S: now also J103.13 (Pin_13), U101.57 (S)
- net DISP_10: now reaches J104.10 (Pin_10)
- net DISP_10: now also FB109.2
- net LD1: now reaches J104.11 (Pin_11)
- net LD1: now also J103.6 (Pin_6), U101.50 (LD1)
- net DISP_12: now reaches J104.12 (Pin_12)
- net DISP_12: now also R114.1
- net CP: now reaches J104.13 (Pin_13)
- net CP: now also J103.11 (Pin_11), U101.53 (CP)
- net DISP_14: now reaches J104.14 (Pin_14)
- net DISP_14: now also R111.2
- net FR: now reaches J104.15 (Pin_15)
- net FR: now also D106.2 (A), J103.7 (Pin_7), U101.56 (FR)
- net VDD: now reaches J104.2 (Pin_2)
- net VDD: now also C101.1, C112.1, C116.1, C120.2, C121.1, D101.1 (K), FB106.1, FB106.2, FB110.1, FB110.2, FB112.1, FB112.2, FB113.1, FB113.2, J103.17 (Pin_17), Q101.1 (E), R108.2, R116.1, R120.1, R124.2, R126.1, R127.1, U102.26 (CE2), U102.28 (VCC), U103.28 (VCC), U104.6 (V+), U105.4 (V+), U108.14 (VCC), U109.14 (VCC), U110.16 (VCC), U111.32 (VCC), C12.1, U113.4 (V+)
- net CPG: now reaches J104.3 (Pin_3)
- net CPG: now also J103.8 (Pin_8), U101.52 (CPG)
- net DISP_4: now reaches J104.4 (Pin_4)
- net DISP_4: now also C110.2
- net CPL: now reaches J104.5 (Pin_5)
- net CPL: now also J103.12 (Pin_12), U101.55 (CPL)
- net DISP_6: now reaches J104.6 (Pin_6)
- net DISP_6: now also R119.2, U105.8, U106.6, U113.8
- net ST: now reaches J104.7 (Pin_7)
- net ST: now also J103.10 (Pin_10), U101.54 (ST)
- net DISP_8: now reaches J104.8 (Pin_8)
- net DISP_8: now also FB108.2
- net LD0: now reaches J104.9 (Pin_9)
- net LD0: now also J103.9 (Pin_9), U101.51 (LD0)
- net at R122.1: now also R120.2, R123.1
- net at R122.2: now also R123.2, R131.1, U105.9 (-), U113.9 (-)
- net +BATT: now reaches C115.1
- net +BATT: now also D101.2 (A), D102.2 (A), J103.16 (Pin_16), Q101.3 (C), R106.1, U106.14 (V_{DD}), U107.14 (V_{DD})
- net at C102.1: now also R110.1
- net VOICE_OUT: now reaches C102.2
- net VOICE_OUT: now also C105.2, J108.6 (Pin_6), R130.1
- net MA0: now reaches U102.10 (A0)
- net MA0: now also U101.34 (MA0)
- net MD0: now reaches U102.11 (I/O0)
- net MD0: now also U101.33 (MD0)
- net MD1: now reaches U102.12 (I/O1)
- net MD1: now also U101.31 (MD1)
- net MD2: now reaches U102.13 (I/O2)
- net MD2: now also U101.30 (MD2)
- net MD3: now reaches U102.15 (I/O3)
- net MD3: now also U101.29 (MD3)
- net MD4: now reaches U102.16 (I/O4)
- net MD4: now also U101.28 (MD4)
- net MD5: now reaches U102.17 (I/O5)
- net MD5: now also U101.27 (MD5)
- net MD6: now reaches U102.18 (I/O6)
- net MD6: now also U101.26 (MD6)
- net MD7: now reaches U102.19 (I/O7)
- net MD7: now also U101.25 (MD7)
- net MA12: now reaches U102.2 (A12)
- net MA12: now also U101.42 (MA12)
- net ~{MCS}: now reaches U102.20 (~{CE1})
- net ~{MCS}: now also U101.43 (~{MCS})
- net MA10: now reaches U102.21 (A10)
- net MA10: now also U101.44 (MA10)
- net ~{MRD}: now reaches U102.22 (~{OE})
- net ~{MRD}: now also U101.45 (~{MRD})
- net MA11: now reaches U102.23 (A11)
- net MA11: now also U101.46 (MA11)
- net MA9: now reaches U102.24 (A9)
- net MA9: now also U101.47 (MA9)
- net MA8: now reaches U102.25 (A8)
- net MA8: now also U101.48 (MA8)
- net ~{MWR}: now reaches U102.27 (~{WE})
- net ~{MWR}: now also U101.49 (~{MWR})
- net MA7: now reaches U102.3 (A7)
- net MA7: now also U101.41 (MA7)
- net MA6: now reaches U102.4 (A6)
- net MA6: now also U101.40 (MA6)
- net MA5: now reaches U102.5 (A5)
- net MA5: now also U101.39 (MA5)
- net MA4: now reaches U102.6 (A4)
- net MA4: now also U101.38 (MA4)
- net MA3: now reaches U102.7 (A3)
- net MA3: now also U101.37 (MA3)
- net MA2: now reaches U102.8 (A2)
- net MA2: now also U101.36 (MA2)
- net MA1: now reaches U102.9 (A1)
- net MA1: now also U101.35 (MA1)
- net at R114.2: now also C107.2
- net RAM_~{CS}: now reaches D108.1 (K)
- net RAM_~{CS}: now also D107.1 (K), J102.29 (Pin_29), R128.1
- net at R116.2: now also C111.1, R109.2, U105.3 (+), U105.5 (+), U113.3 (+), U113.5 (+)
- net P14: now reaches R108.1
- net P14: now also R107.1, R127.2, U101.63 (P14), U109.1
- net at R101.1: now also Q101.2 (B)
- net POWER_EN: now reaches R101.2
- net POWER_EN: now also J103.25 (Pin_25)
- net P15: now reaches R126.2
- net P15: now also U101.62 (P15), U109.5
- net ~{RES}: now reaches D106.1 (K)
- net ~{RES}: now also D104.1 (K), J103.15 (Pin_15), U110.1 (~{Mr})
- net SO1: now reaches U101.60 (SO1)
- net SO1: now also C106.2
- net VIN: now reaches U101.61 (VIN)
- net P13: now reaches U101.64 (P13)
- net P13: now also J107.2 (Pin_2)
- net P12: now reaches U101.65 (P12)
- net P12: now also J107.1 (Pin_1)
- net P11: now reaches U101.66 (P11)
- net P11: now also J107.3 (Pin_3)
- net P10: now reaches U101.67 (P10)
- net P10: now also J107.4 (Pin_4)
- net SCK: now reaches U101.68 (SCK)
- net SCK: now also FB105.2
- net SIN: now reaches U101.69 (SIN)
- net SIN: now also FB104.2
- net SOUT: now reaches U101.70 (SOUT)
- net SOUT: now also FB103.2
- net at U101.73 (CK2): now also TP102.1
- net at U101.74 (CK1): now also C117.1
- net PHI: now reaches U101.75 (PHI)
- net at FB105.1: now also R105.1
- net EDGE_14: now reaches C108.1
- net EDGE_14: now also C118.1, C119.2, J103.14 (Pin_14), R121.1, U104.3 (+)
- net at R129.1: now also J108.4 (Pin_4)
- net at R129.2: now also J108.5 (Pin_5)
- net at R111.1: now also C104.2
- net at RV101.1: now also R131.2
- net P15_MEMCARD_EXT: now reaches U109.6
- net P15_MEMCARD_EXT: now also J107.6 (Pin_6)
- net at D102.1 (K): now also D103.2 (A)
- net P14_EDGE: now reaches R107.2
- net P14_EDGE: now also J103.4 (Pin_4)
- net at C105.1: now also R115.1
- net SOUT_EDGE: now reaches U106.1
- net SOUT_EDGE: now also J103.3 (Pin_3)
- net LNK_EDGE_EN: now reaches U106.13
- net LNK_EDGE_EN: now also J103.20 (Pin_20), U106.12, U106.5
- net at U106.2: now also R103.2, U107.1
- net at R103.1: now also FB103.1
- net LNK_EN: now reaches U107.13
- net LNK_EN: now also D104.2 (A), D105.2 (A), R106.2, U107.12, U107.5
- net EDGE_26(SOUT): now reaches U107.2
- net EDGE_26(SOUT): now also J103.26 (Pin_26)
- net EDGE_19: now reaches U106.8
- net EDGE_19: now also J103.19 (Pin_19)
- net EDGE_18: now reaches U106.9
- net EDGE_18: now also J103.18 (Pin_18)
- net at FB109.1: now also J106.5 (Pin_5)
- net at D103.1 (K): now also J108.7 (Pin_7)
- net at FB104.1: now also R104.1
- net SRA16: now reaches U111.2 (A16)
- net SRA16: now also U110.5 (Q1)
- net SR~{CE}: now reaches U111.22 (~{CE})
- net SR~{CE}: now also U108.6
- net SRA15: now reaches U111.3 (A15)
- net SRA15: now also U110.2 (Q0)
- net SRA17: now reaches U111.30 (A17)
- net SRA17: now also U110.7 (Q2)
- net SRA18: now reaches U111.31 (A18)
- net SRA18: now also U110.10 (Q3)
- net EDGE_23: now reaches J108.2 (Pin_2)
- net EDGE_23: now also J103.23 (Pin_23)
- net EDGE_22: now reaches J108.3 (Pin_3)
- net EDGE_22: now also J103.22 (Pin_22)
- net at C110.1: now also U104.5
- net XTAL_2: now reaches Y101.1
- net XTAL_2: now also C114.1, J103.30 (Pin_30), R102.2, TP101.1
- net at R117.1: now also R118.1, R119.1, U105.10 (+), U113.10 (+)
- net at C106.1: now also R133.1
- net at R105.2: now also U106.10, U107.11
- net SCK_EDGE: now reaches U106.11
- net SCK_EDGE: now also J103.5 (Pin_5)
- net EDGE_21: now reaches D105.1 (K)
- net EDGE_21: now also J103.21 (Pin_21)
- net EDGE_27(SIN): now reaches U107.3
- net EDGE_27(SIN): now also J103.27 (Pin_27)
- net at U107.4: now also R104.2, U106.3
- net at FB108.1: now also J106.4 (Pin_4)
- net at D110.2 (A): now also D109.1 (K)
- net at U108.4: now also U108.11
- net at U108.5: now also U108.10, U108.3
- net at R115.2: now also R113.1, R133.2
- net at J106.1 (Pin_1): now also C118.2
- net at J106.3 (Pin_3): now also C119.1
- net at R118.2: now also D109.2 (A), R124.1
- net SIN_EDGE: now reaches U106.4
- net SIN_EDGE: now also J103.2 (Pin_2)
- net P14_MEMCARD_EXT: now reaches J107.5 (Pin_5)
- net P14_MEMCARD_EXT: now also U109.3
- net USE_CART: now reaches U108.12
- net USE_CART: now also J103.24 (Pin_24), U108.13, U108.9
- net at R113.2: now also C107.1, U105.7, U113.7
- net at C109.1: now also U104.7 (BYPASS)
- net A15': now reaches U108.8
- net A15': now also J101.21 (Pin_21)
- net EDGE_28(SCK): now reaches J103.28 (Pin_28)
- net EDGE_31: now reaches J103.31 (Pin_31)
- no-connect marks 0 -> 1
Other:
- note added: "SYSROM/CART_Switch"
- moved on the sheet: C102, C103, C104, C105, C106, C107, C108, C109, C110, C112, C113, C114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
