File: Hardware/Main-Board/Main-Board.kicad_sch (KiCad schematic)
At the start: 103 parts, among them J101 ProgrammCard, J102 MemoryCard, J103 Edge_Connector, J104 LCD_CON, J106 EXT_AUDIO, J107 MOUSE_PORT, J108 Voice_Board_Mock, Q101 C9012, U101 DMG CPU, U102 GM76C88LFW-15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

Commit message: Fixed error in Audio-Mixer - Added more signal names
Connections:
- net LNK_EDGE_EN: no longer J103.20 (Pin_20)
- net MC_?_4: now also R113.1, R115.2, R133.2
- net DISP_10 renamed ADUIO_OUT_2'
- net DISP_12 renamed AUDIO_OUT_1
- net DISP_14 renamed ADUIO_OUT_2
- net ADUIO_OUT_2: no longer R111.2
- net DISP_4 renamed SPEAKER
- net DISP_6 renamed BATT_LOW
- net DISP_8 renamed ADUIO_OUT_1'
- net ADUIO_OUT_1': no longer J104.8 (Pin_8)
- net EDGE_14 renamed MONO_IN
- net EDGE_21 renamed LNK_ASIC_EN
- net EDGE_22 renamed VOICE_DATA
- net EDGE_23 renamed VOICE_~{RST}
- net LNK_EN renamed LNK_ASIC_EN'
- net P14_EDGE renamed P14_EXT
- new net AUDIO_OUT_1': J104.8 (Pin_8)
- new net AUDIO_OUT_2: R111.2
- new net LNK_EXT_EN: J103.20 (Pin_20)
Other:
- moved on the sheet: C102, C103, C104, C105, C106, C107, C112, D109, D110, R109, R110, R111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
